File: kicad-pps.kicad_pcb (KiCad board)
At the start: 2 copper layers, 100 x 100 mm, 46 parts, among them J1 Conn_01x01_Pin, J10 Conn_01x01_Pin, J14 Screw_Terminal_2_P5.00mm, J15 Conn_01x01_Pin, J16 Conn_01x01_Pin, J17 Conn_01x01_Pin, J3 Conn_01x01_Pin, J4 Screw_Terminal_2_P5.00mm, J5 Screw_Terminal_2_P5.00mm, J6 Screw_Terminal_01x04, J7 AudioJack4, J8 AudioJack4, J9 AudioJack4, U3 MCP4131-xxxx-P, U4 MCP4131-xxxx-P, U5 MCP4131-xxxx-P, U6 LMV324, U7 LMV324

Commit message: initial fran commit
Parts:
- R11: value 820 -> 820k
- R14: value R -> 3.3k
- R15, R16: value R -> 10k
Connections:
- R21 pad 1: Net-(U7D-+) -> Net-(U7D--)
- R22 pad 2: Net-(U7D-+) -> Net-(U7D--)
- U7 pad 12: Net-(U7D-+) -> /+1V65
- U7 pad 13: /+1V65 -> Net-(U7D--)
Routing:
- net Net-(U7D-+): track 46.5 -> 0.00 mm
- net /+1V65: track 280.1 -> 326.6 mm
- net /SPI_SCK: track 165.5 -> 166.5 mm
- net GND: track 217.6 -> 218.2 mm

Commit message: Version 2: Bicapa
Parts:
- added C18: 100n, Capacitor_THT:CP_Radial_Tantal_D5.5mm_P2.50mm, F.Cu at (88.1, 72.6)
- added J11: Conn_01x01_Pin, Connector_PinHeader_2.54mm:PinHeader_1x01_P2.54mm_Vertical, F.Cu at (200.9, 43.5)
- added J12: Conn_01x01_Pin, Connector_PinHeader_2.54mm:PinHeader_1x01_P2.54mm_Vertical, F.Cu at (205.5, 38.9)
- added J13: Conn_01x01_Pin, Connector_PinHeader_2.54mm:PinHeader_1x01_P2.54mm_Vertical, F.Cu at (205.5, 43.5)
- added J18: Conn_01x01_Pin, Connector_PinHeader_2.54mm:PinHeader_1x01_P2.54mm_Vertical, F.Cu at (210.1, 43.5)
- added J19: Conn_01x05_Pin, Connector_PinHeader_2.54mm:PinHeader_1x05_P2.54mm_Vertical, F.Cu at (200.9, 48.1)
- added J2: Conn_01x05_Pin, Connector_PinHeader_2.54mm:PinHeader_1x05_P2.54mm_Horizontal, F.Cu at (160.5, 52.3)
- added J20: Conn_01x05_Pin, Connector_PinHeader_2.54mm:PinHeader_1x05_P2.54mm_Vertical, F.Cu at (206.0, 48.5)
- added JP1: Jumper_2_Bridged, TestPoint:TestPoint_2Pads_Pitch2.54mm_Drill0.8mm, F.Cu at (184.9, 31.0)
- added JP2: Jumper_2_Bridged, TestPoint:TestPoint_2Pads_Pitch2.54mm_Drill0.8mm, F.Cu at (184.2, 35.5)
- added JP3: Jumper_2_Bridged, TestPoint:TestPoint_2Pads_Pitch2.54mm_Drill0.8mm, F.Cu at (184.2, 38.8)
- added JP4: Jumper_2_Bridged, TestPoint:TestPoint_2Pads_Pitch2.54mm_Drill0.8mm, F.Cu at (184.2, 42.2)
- added JP5: Jumper_2_Bridged, TestPoint:TestPoint_2Pads_Pitch2.54mm_Drill0.8mm, F.Cu at (184.2, 45.5)
- added JP6: Jumper_2_Bridged, TestPoint:TestPoint_2Pads_Pitch2.54mm_Drill0.8mm, F.Cu at (184.2, 48.9)
- J14, J5: value Screw_Terminal_2_P5.00mm -> Conn_01x01_Pin; footprint TerminalBlock:TerminalBlock_MaiXu_MX126-5.0-02P_1x02_P5.00mm -> Connector_PinHeader_2.54mm:PinHeader_1x01_P2.54mm_Vertical
- J4: value Screw_Terminal_2_P5.00mm -> Conn_01x05_Pin; footprint Connector_PinHeader_2.54mm:PinHeader_1x02_P2.54mm_Vertical -> Connector_PinHeader_2.54mm:PinHeader_1x05_P2.54mm_Horizontal
- moved J14 124.1 mm to (210.1, 38.9), turned to 0 degrees
- moved J4 84.7 mm to (82.0, 36.1), turned to 90 degrees
- moved C17 52.6 mm to (145.8, 62.7), turned to 180 degrees
- moved J5 44.3 mm to (200.9, 38.9), turned to 0 degrees
- moved J6 5.84 mm to (78.5, 41.7)
- moved R11 1.96 mm to (84.8, 43.5)
- moved R12 1.96 mm to (84.8, 50.0)
- moved R13 1.96 mm to (84.8, 57.0)
- moved J8 1.76 mm to (78.0, 115.3)
- moved J7 1.55 mm to (78.0, 76.0)
- moved J9 1.46 mm to (78.0, 95.7)
- moved C15 1.39 mm to (159.5, 45.0)
- turned R10 to -115 degrees
Connections:
- A1 pad 21: unconnected-(A1-VBAT-Pad21) -> +5V
- A1 pad 31: unconnected-(A1-MISO1/PA6-Pad31) -> /+1V65
- C17 pad 1: +3V3 -> +5V
- J14 pad 1: /AC_NEU -> unconnected-(J14-Pin_1-Pad1)
- J4 pad 1: /TX_UART -> /AC_PH1
- J4 pad 2: /RX_UART -> /AC_PH1
- J5 pad 1: +3V3 -> unconnected-(J5-Pin_1-Pad1)
- J7 pad R1: (no net) -> unconnected-(J7-PadR1)
- J7 pad R2: (no net) -> unconnected-(J7-PadR2)
- J7 pad S: (no net) -> /+1V65
- J7 pad T: (no net) -> /AC_C1
- J8 pad R1: (no net) -> unconnected-(J8-PadR1)
- J8 pad R2: (no net) -> unconnected-(J8-PadR2)
- J8 pad S: (no net) -> /+1V65
- J8 pad T: (no net) -> /AC_C3
- J9 pad R1: (no net) -> unconnected-(J9-PadR1)
- J9 pad R2: (no net) -> unconnected-(J9-PadR2)
- J9 pad S: (no net) -> /+1V65
- J9 pad T: (no net) -> /AC_C2
Routing:
- net Net-(U7D--): track 0.00 -> 45.3 mm
- net /+1V65: track 326.6 -> 354.1 mm
- net +5V: track 0.00 -> 26.7 mm
- net +3V3: track 197.6 -> 173.6 mm, vias 9 -> 5
- net /ADC1_CH0: track 96.1 -> 76.5 mm, vias 0 -> 2
- net /TX_UART: track 47.7 -> 40.7 mm
- net /RX_UART: track 39.2 -> 33.5 mm
- net /AC_PH3: track 11.3 -> 7.04 mm
- net /SPI_SCK: track 166.5 -> 170.4 mm
- net /AC_PH2: track 10.4 -> 6.96 mm
- net GND: track 218.2 -> 215.5 mm
- net /SPI_MOSI: track 173.3 -> 175.9 mm
- net Net-(R11-Pad2): track 17.5 -> 15.9 mm
- net Net-(R12-Pad2): track 9.35 -> 7.87 mm
- net /AC_C1: track 55.7 -> 57.1 mm
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- added copper zone on F.Cu, net GND

Commit message: branch completo-bicapa
Parts:
- removed J19, J20: Conn_01x05_Pin, Connector_PinHeader_2.54mm:PinHeader_1x05_P2.54mm_Vertical
- removed J4: Conn_01x05_Pin, Connector_PinHeader_2.54mm:PinHeader_1x05_P2.54mm_Horizontal
- added C1: 100n, Capacitor_THT:CP_Radial_Tantal_D5.5mm_P2.50mm, F.Cu at (110.7, 65.0)
- added C2: 10u, Capacitor_THT:CP_Radial_D6.3mm_P2.50mm, F.Cu at (110.7, 69.9)
- added F1: Fuse, Fuse:Fuseholder_Clip-5x20mm_Littelfuse_445-030_Inline_P20.50x5.20mm_D1.30mm_Horizontal, F.Cu at (79.3, 137.7)
- added RV1: Varistor, Varistor:RV_Disc_D12mm_W3.9mm_P7.5mm, F.Cu at (79.3, 109.5)
- added U1: HLK-5M05, Converter_ACDC:Converter_ACDC_Hi-Link_HLK-5Mxx, F.Cu at (86.4, 100.4)
- added U2: ESP32-C3-SuperMini, esp32-c3-supermini:ESP32-C3-SuperMini, F.Cu at (128.8, 66.5)
- J2: value Conn_01x05_Pin -> Conn_01x12_Pin; footprint Connector_PinHeader_2.54mm:PinHeader_1x05_P2.54mm_Horizontal -> Connector_PinHeader_2.54mm:PinHeader_1x12_P2.54mm_Vertical
- R12: value 820 -> 820k
- R13: value R -> 820k
- R17, R20: value R -> 3.3k
- R18, R19, R22: value R -> 10k
- R21: value 820 -> 10k
- U6, U7: moved to F.Cu
- moved H2 144.2 mm to (216.6, 57.1)
- moved J9 133.0 mm to (200.2, 148.3), turned to 180 degrees
- moved J12 129.0 mm to (138.9, 149.4)
- moved JP3 121.9 mm to (132.7, 149.4)
- moved J7 112.8 mm to (164.6, 148.3), turned to 180 degrees
- moved J8 109.5 mm to (182.4, 148.3), turned to 180 degrees
- moved U5 108.7 mm to (201.4, 115.6)
- moved R8 107.6 mm to (200.2, 135.3)
- moved JP2 107.2 mm to (132.7, 129.5)
- moved J11 106.1 mm to (138.9, 129.5)
- moved J6 104.3 mm to (88.0, 145.5), turned to 0 degrees
- moved J17 96.8 mm to (187.3, 102.0), turned to -90 degrees
- moved R11 94.2 mm to (88.0, 137.7), turned to 90 degrees
- moved J14 93.3 mm to (192.5, 130.6)
- moved JP1 93.2 mm to (132.7, 108.2), turned to 0 degrees
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Connections:
- A1 pad 14: /TX_UART -> Net-(A1-PB6/SCL1/TX1)
- A1 pad 15: /RX_UART -> Net-(A1-PB7/SDA1/RX1)
- A1 pad 20: +3V3 -> unconnected-(A1-3V3-Pad20)
- J11 pad 1: unconnected-(J11-Pin_1-Pad1) -> Net-(J11-Pin_1)
- J12 pad 1: unconnected-(J12-Pin_1-Pad1) -> Net-(J12-Pin_1)
- J13 pad 1: unconnected-(J13-Pin_1-Pad1) -> Net-(J13-Pin_1)
- J14 pad 1: unconnected-(J14-Pin_1-Pad1) -> Net-(J14-Pin_1)
- J18 pad 1: unconnected-(J18-Pin_1-Pad1) -> Net-(J18-Pin_1)
- J2 pad 1: +5V -> GND
- J2 pad 2: /TX_UART -> GND
- J2 pad 3: /RX_UART -> GND
- J5 pad 1: unconnected-(J5-Pin_1-Pad1) -> Net-(J5-Pin_1)
- J6 pad 1: /AC_NEU -> /AC_PH1
- J6 pad 2: /AC_PH1 -> /AC_PH2
- J6 pad 3: /AC_PH2 -> /AC_PH3
- J6 pad 4: /AC_PH3 -> GNDPWR
- JP1 pad 1: unconnected-(JP1-A-Pad1) -> Net-(JP1-A)
- JP1 pad 2: unconnected-(JP1-B-Pad2) -> Net-(J5-Pin_1)
- JP2 pad 1: unconnected-(JP2-A-Pad1) -> Net-(JP2-A)
- JP2 pad 2: unconnected-(JP2-B-Pad2) -> Net-(J11-Pin_1)
- JP3 pad 1: unconnected-(JP3-A-Pad1) -> Net-(JP3-A)
- JP3 pad 2: unconnected-(JP3-B-Pad2) -> Net-(J12-Pin_1)
- JP4 pad 1: unconnected-(JP4-A-Pad1) -> /AC_C1
- JP4 pad 2: unconnected-(JP4-B-Pad2) -> Net-(J13-Pin_1)
- JP5 pad 1: unconnected-(JP5-A-Pad1) -> /AC_C3
- JP5 pad 2: unconnected-(JP5-B-Pad2) -> Net-(J14-Pin_1)
- JP6 pad 1: unconnected-(JP6-A-Pad1) -> /AC_C2
- JP6 pad 2: unconnected-(JP6-B-Pad2) -> Net-(J18-Pin_1)
- R14 pad 2: Net-(R14-Pad2) -> Net-(JP1-A)
- R15 pad 2: Net-(R14-Pad2) -> Net-(J5-Pin_1)
- R17 pad 2: Net-(R17-Pad2) -> Net-(JP2-A)
- R18 pad 2: Net-(R17-Pad2) -> Net-(J11-Pin_1)
- R20 pad 2: Net-(R20-Pad2) -> Net-(JP3-A)
- R21 pad 2: Net-(R20-Pad2) -> Net-(J12-Pin_1)
- TR1 pad 2: /AC_NEU -> GNDPWR
- TR1 pad 4: Net-(R14-Pad2) -> Net-(JP1-A)
- TR2 pad 2: /AC_NEU -> GNDPWR
- TR2 pad 4: Net-(R17-Pad2) -> Net-(JP2-A)
- TR3 pad 2: /AC_NEU -> GNDPWR
- TR3 pad 4: Net-(R20-Pad2) -> Net-(JP3-A)
- U3 pad 5: /ADC2_CH5 -> Net-(J13-Pin_1)
- U3 pad 7: /AC_C1 -> /ADC2_CH5
- U4 pad 5: /AC_C3 -> Net-(J14-Pin_1)
- U5 pad 5: /ADC2_CH3 -> Net-(J18-Pin_1)
- U5 pad 7: /AC_C2 -> /ADC2_CH3
Routing:
- net GND: track 215.5 -> 70.4 mm, vias 6 -> 3
- net /AC_NEU: track 89.8 -> 0.00 mm
- net Net-(A1-PB6/SCL1/TX1): track 0.00 -> 72.8 mm
- net Net-(A1-PB7/SDA1/RX1): track 0.00 -> 72.3 mm
- net /+1V65: track 354.1 -> 421.6 mm, vias 2 -> 3
- net +5V: track 26.7 -> 88.8 mm
- net /AC_C3: track 70.6 -> 10.2 mm
- net /SPI_CS5: track 23.9 -> 77.6 mm
- net /AC_C1: track 57.1 -> 10.2 mm
- net Net-(R11-Pad2): track 15.9 -> 57.5 mm
- net /TX_UART: track 40.7 -> 0.00 mm
- net /SPI_CS3: track 95.1 -> 54.7 mm
- net Net-(U3-P0W): track 10.9 -> 50.9 mm
- net /ADC2_CH3: track 107.5 -> 68.3 mm, vias 2 -> 0
- net +3V3: track 173.6 -> 210.2 mm, vias 5 -> 8
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- added copper zone on B.Cu, net GND
- added copper zone on B.Cu, net GNDPWR
- removed copper zone on F.Cu, net GND
Other:
- board size 100 x 100 mm -> 150 x 100 mm

Commit message: branch completo-unicapa wip
Parts:
- removed C17: 100n, Capacitor_THT:CP_Radial_Tantal_D5.5mm_P2.50mm
- J1, J10, J15, J16, J17, J3, U6, U7: moved to B.Cu
- moved R10 36.8 mm to (215.4, 75.7), turned to 90 degrees
- moved U3 36.1 mm to (201.9, 116.0)
- moved J13 36.1 mm to (210.8, 130.5)
- moved J7 36.1 mm to (200.7, 148.3)
- moved JP4 36.1 mm to (200.7, 130.5)
- moved R6 36.1 mm to (200.7, 135.3)
- moved U5 35.7 mm to (165.7, 116.0)
- moved J18 35.7 mm to (174.6, 130.5)
- moved J9 35.7 mm to (164.5, 148.3)
- moved JP6 35.7 mm to (164.5, 130.5)
- moved R8 35.7 mm to (164.5, 135.3)
- moved C1 33.8 mm to (143.8, 57.7), turned to -90 degrees
- moved C2 33.3 mm to (143.8, 65.5)
- moved R9 20.3 mm to (215.5, 89.4), turned to 90 degrees
- moved J15 20.3 mm to (189.5, 81.8), turned to 180 degrees
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Connections:
- A1 pad 19: GND -> unconnected-(A1-GND-Pad19)
- U5 pad 5: Net-(J18-Pin_1) -> /ADC2_CH3
- U5 pad 7: /ADC2_CH3 -> Net-(J18-Pin_1)
Routing:
- net +3V3: track 210.2 -> 0.00 mm, vias 8 -> 0
- net /SPI_MOSI: track 165.6 -> 0.00 mm
- net /SPI_SCK: track 164.9 -> 0.00 mm
- net /+1V65: track 421.6 -> 265.2 mm, vias 3 -> 0
- net /SPI_CS5: track 77.6 -> 0.00 mm
- net /ADC2_CH5: track 88.0 -> 15.2 mm
- net GND: track 70.4 -> 0.06 mm, vias 3 -> 0
- net /SPI_CS4: track 62.0 -> 0.00 mm
- net /ADC1_CH2: track 87.1 -> 28.5 mm
- net /SPI_CS3: track 54.7 -> 0.00 mm
- net Net-(U3-P0W): track 50.9 -> 0.00 mm
- net Net-(U4-P0W): track 39.3 -> 0.00 mm
- net Net-(U7C-+): track 38.6 -> 0.00 mm
- net /ADC2_CH3: track 68.3 -> 32.4 mm
- net Net-(U7D--): track 48.5 -> 12.7 mm
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
Commit message: completo unicapa
Parts:
- added C19: 100n, Capacitor_THT:CP_Radial_Tantal_D5.5mm_P2.50mm, F.Cu at (171.5, 83.6)
- added J19: Conn_01x03_Pin, Connector_PinHeader_2.54mm:PinHeader_1x03_P2.54mm_Vertical, F.Cu at (161.2, 123.6)
- added J20: Conn_01x03_Pin, Connector_PinHeader_2.54mm:PinHeader_1x03_P2.54mm_Vertical, F.Cu at (149.0, 76.2)
- added J4: Conn_01x03_Pin, Connector_PinHeader_2.54mm:PinHeader_1x03_P2.54mm_Vertical, F.Cu at (149.6, 101.4)
- J1, J10, J15, J16, J17, J3: moved to F.Cu
- J2: value Conn_01x12_Pin -> Conn_01x03_Pin; footprint Connector_PinHeader_2.54mm:PinHeader_1x12_P2.54mm_Vertical -> Connector_PinHeader_2.54mm:PinHeader_1x03_P2.54mm_Vertical
- moved R10 48.7 mm to (168.3, 88.0), turned to -90 degrees
- moved R9 43.8 mm to (172.6, 98.2)
- moved C1 32.6 mm to (111.1, 57.4)
- moved C2 32.6 mm to (111.1, 65.3)
- moved J2 29.6 mm to (199.4, 84.8)
- moved C16 19.0 mm to (203.0, 81.8), turned to 0 degrees
- moved TR3 12.6 mm to (113.6, 129.9), turned to 0 degrees
- moved TR2 12.1 mm to (113.6, 110.2), turned to 0 degrees
- moved TR1 11.7 mm to (113.6, 90.4), turned to 0 degrees
- moved J1 11.4 mm to (158.6, 81.9), turned to 180 degrees
- moved J10 11.4 mm to (163.5, 96.9), turned to 180 degrees
- moved J3 11.4 mm to (158.6, 96.9), turned to 180 degrees
- moved U7 11.4 mm to (161.0, 89.8)
- moved J7 8.90 mm to (209.6, 148.3)
- moved J8 6.88 mm to (189.4, 148.3)
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Connections:
- A1 pad 18: unconnected-(A1-5V-Pad18) -> +5V
- A1 pad 21: +5V -> unconnected-(A1-VBAT-Pad21)
- A1 pad 33: /SPI_CS5 -> /SPI_CS3
- A1 pad 35: /SPI_CS3 -> /SPI_CS5
- U5 pad 5: /ADC2_CH3 -> Net-(J18-Pin_1)
- U5 pad 7: Net-(J18-Pin_1) -> /ADC2_CH3
Routing:
- net GND: track 0.06 -> 557.5 mm
- net /SPI_MOSI: track 0.00 -> 165.1 mm, vias 0 -> 2
- net /SPI_SCK: track 0.00 -> 164.7 mm, vias 0 -> 2
- net +3V3: track 0.00 -> 162.6 mm, vias 0 -> 12
- net GNDPWR: track 0.00 -> 153.6 mm
- net /+1V65: track 265.2 -> 385.7 mm, vias 0 -> 13
- net Net-(U7D--): track 12.7 -> 78.5 mm, vias 0 -> 2
- net /SPI_CS3: track 0.00 -> 55.0 mm, vias 0 -> 4
- net /ADC1_CH2: track 28.5 -> 80.1 mm
- net Net-(U3-P0W): track 0.00 -> 44.2 mm
- net /ADC2_CH5: track 15.2 -> 57.3 mm
- net /SPI_CS4: track 0.00 -> 41.8 mm, vias 0 -> 4
- net /SPI_CS5: track 0.00 -> 39.2 mm, vias 0 -> 2
- net /ADC1_CH1: track 30.2 -> 64.3 mm
- net Net-(U5-P0W): track 0.00 -> 34.0 mm
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- removed copper zone on B.Cu, net GNDPWR

Commit message: mejoras
Parts:
- added J21: Conn_01x02_Pin, Connector_Molex:Molex_KK-396_5273-02A_1x02_P3.96mm_Vertical, F.Cu at (68.1, 33.3)
- added J22: Conn_01x03_Pin, Connector_PinHeader_2.54mm:PinHeader_1x03_P2.54mm_Vertical, F.Cu at (112.6, 28.3)
- moved C2 72.4 mm to (48.1, 29.7), turned to 180 degrees
- moved C1 61.8 mm to (55.9, 29.7), turned to 180 degrees
- moved R13 54.2 mm to (62.3, 99.3)
- moved R11 54.2 mm to (47.3, 99.4)
- moved R12 54.2 mm to (54.8, 99.4)
- moved J6 53.6 mm to (47.6, 107.3)
- moved U2 49.6 mm to (87.6, 38.8)
- moved J13 49.0 mm to (169.1, 102.8)
- moved J14 49.0 mm to (149.0, 102.8)
- moved J18 49.0 mm to (129.0, 102.8)
- moved JP4 49.0 mm to (159.0, 102.8)
- moved JP5 49.0 mm to (138.9, 102.8)
- moved JP6 49.0 mm to (118.8, 102.8)
- moved A1 49.0 mm to (144.5, 39.4)
- moved C15 49.0 mm to (105.9, 80.3)
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Connections:
- A1 pad 19: unconnected-(A1-GND-Pad19) -> GND
- J6 pad 1: /AC_PH1 -> GNDPWR
- J6 pad 2: /AC_PH2 -> /AC_PH1
- J6 pad 3: /AC_PH3 -> /AC_PH2
- J6 pad 4: GNDPWR -> /AC_PH3
Routing:
- net GND: track 557.5 -> 698.6 mm
- net Net-(A1-PB6/SCL1/TX1): track 70.4 -> 89.5 mm, vias 0 -> 2
- net +5V: track 91.1 -> 105.3 mm, vias 2 -> 0
- net Net-(A1-PB7/SDA1/RX1): track 63.4 -> 72.5 mm, vias 0 -> 2
- net GNDPWR: track 153.6 -> 145.5 mm
- net Net-(R11-Pad2): track 45.2 -> 37.2 mm
- net Net-(R12-Pad2): track 26.5 -> 21.1 mm
- net Net-(R13-Pad2): track 12.7 -> 17.7 mm
- net Net-(U4-P0W): track 33.2 -> 34.8 mm
- net /AC_PH1: track 24.5 -> 26.0 mm
- net /AC_PH3: track 9.56 -> 8.10 mm
- net /AC_PH2: track 8.40 -> 9.00 mm
- net /ADC2_CH5: track 57.3 -> 57.8 mm

Commit message: fixes
Connections:
- net GNDPWR renamed /AC_NEU
- net VAC renamed Net-(U1-AC/L)
Routing:
- net Net-(U4-P0W): track 34.8 -> 37.3 mm
- net +3V3: track 162.9 -> 161.5 mm
- net Net-(J18-Pin_1): track 28.7 -> 29.8 mm, vias 2 -> 1
- net /ADC2_CH4: track 44.5 -> 45.4 mm
- net GND: vias 0 -> 1
- added copper zone on F.Cu, net GND
