File: kicad-pps.kicad_pcb (KiCad board)
At the start: 2 copper layers, 150 x 100 mm, 68 parts, among them J1 Conn_01x01_Pin, J10 Conn_01x01_Pin, J11 Conn_01x01_Pin, J12 Conn_01x01_Pin, J13 Conn_01x01_Pin, J14 Conn_01x01_Pin, J15 Conn_01x01_Pin, J16 Conn_01x01_Pin, J17 Conn_01x01_Pin, J18 Conn_01x01_Pin, J19 Conn_01x03_Pin, J2 Conn_01x03_Pin, J20 Conn_01x03_Pin, J21 Conn_01x02_Pin, J22 Conn_01x03_Pin, J3 Conn_01x01_Pin, J4 Conn_01x03_Pin, J5 Conn_01x01_Pin, J6 Screw_Terminal_01x04, J7 AudioJack4, J8 AudioJack4, J9 AudioJack4, U1 HLK-5M05, U2 ESP32-C3-SuperMini, U3 MCP4131-xxxx-P, U4 MCP4131-xxxx-P, U5 MCP4131-xxxx-P, U6 LMV324, U7 LMV324

Commit message: rev 2
Parts:
- added G***: LOGO, LOGO, B.Cu at (49.6, 65.0)
- added J23: Conn_01x01_Pin, Connector_PinHeader_2.54mm:PinHeader_1x01_P2.54mm_Vertical, F.Cu at (111.1, 54.3)
- J20: value Conn_01x03_Pin -> Conn_01x04_Pin; footprint Connector_PinHeader_2.54mm:PinHeader_1x03_P2.54mm_Vertical -> Connector_PinHeader_2.54mm:PinHeader_1x04_P2.54mm_Vertical
- moved J20 2.00 mm to (106.6, 48.3)
Routing:
- net GND: track 698.6 -> 750.6 mm
- net Net-(J18-Pin_1): track 29.8 -> 24.0 mm, vias 1 -> 2
- net /+1V65: track 385.6 -> 391.2 mm
- net Net-(J14-Pin_1): track 28.1 -> 23.9 mm
- net Net-(U5-P0W): track 34.0 -> 35.3 mm
- net /SPI_MOSI: track 165.1 -> 164.1 mm
- net /SPI_CS4: track 41.8 -> 42.5 mm
- net +3V3: track 161.5 -> 161.6 mm, vias 12 -> 14
Other:
- board text added: "+5V"
- board text added: "1"
- board text added: "2"
- board text added: "3"
- board text added: "C0"
- board text added: "C1"
- board text added: "C2"
- board text added: "C3"
- board text added: "C4"
- board text added: "C5"
- board text added: "C6"
- board text added: "Fabrizio Contigiani Francisco Moglia"
- board text added: "G"
- board text added: "GND"
- board text added: "I1"
- board text added: "I2"
- board text added: "I3"
- board text added: "Medidor de Energía Bidireccional Trifásico"
- board text added: "N"
- board text added: "Plane Connection"
- board text added: "R"
- board text added: "T"
- board text added: "UART"
- board text added: "V1"
- board text added: "V2"
- board text added: "V3"

Commit message: fix pdf
Routing:
- net GND: track 750.6 -> 748.4 mm
