File: kicad-pps.kicad_sch (KiCad schematic)
At the start: 56 parts, among them J1 Conn_01x01_Pin, J10 Conn_01x01_Pin, J11 Conn_01x08_Socket, J12 Conn_01x08_Socket, J13 Screw_Terminal_2_P5.00mm, J14 Screw_Terminal_2_P5.00mm, J15 Conn_01x01_Pin, J16 Conn_01x01_Pin, J17 Conn_01x01_Pin, J3 Conn_01x01_Pin, J4 Screw_Terminal_2_P5.00mm, J5 Screw_Terminal_2_P5.00mm, J6 Screw_Terminal_01x04, J7 AudioJack4, J8 AudioJack4, J9 AudioJack4, U2 AMS1117-3.3, U3 MCP4131-xxxx-P, U4 MCP4131-xxxx-P, U5 MCP4131-xxxx-P, U6 LMV324, U7 LMV324

Commit message: initial fran commit
Parts:
- removed C1, C2: 10u, Capacitor_THT:CP_Radial_D6.3mm_P2.50mm, symbol Device:C_Polarized
- removed C19, C20: 100n, Capacitor_THT:CP_Radial_Tantal_D5.5mm_P2.50mm, symbol Device:C
- removed J11, J12: Conn_01x08_Socket, Connector_PinSocket_2.54mm:PinSocket_1x08_P2.54mm_Vertical, symbol Connector:Conn_01x08_Socket
- removed J13: Screw_Terminal_2_P5.00mm, TerminalBlock:TerminalBlock_MaiXu_MX126-5.0-02P_1x02_P5.00mm, symbol PCM_SL_Screw_Terminal:Screw_Terminal_2_P5.00mm
- removed PS1: HLK-5M05, Converter_ACDC:Converter_ACDC_Hi-Link_HLK-5Mxx, symbol Converter_ACDC:HLK-5M05
- removed U2: AMS1117-3.3, Package_TO_SOT_SMD:SOT-223-3_TabPin2, symbol Regulator_Linear:AMS1117-3.3
- R11: value 820 -> 820k
- R14: value R -> 3.3k
- R15, R16: value R -> 10k
Connections:
- net ADC2_offset: now reaches A1.31 (MISO1/PA6)

Commit message: Version 2: Bicapa
Parts:
- removed J14, J5: Screw_Terminal_2_P5.00mm, TerminalBlock:TerminalBlock_MaiXu_MX126-5.0-02P_1x02_P5.00mm, symbol PCM_SL_Screw_Terminal:Screw_Terminal_2_P5.00mm
- removed J4: Screw_Terminal_2_P5.00mm, Connector_PinHeader_2.54mm:PinHeader_1x02_P2.54mm_Vertical, symbol PCM_SL_Screw_Terminal:Screw_Terminal_2_P5.00mm
- added J11, J12, J13, J14, J18, J5: Conn_01x01_Pin, Connector_PinHeader_2.54mm:PinHeader_1x01_P2.54mm_Vertical, symbol Connector:Conn_01x01_Pin
- added J19, J20: Conn_01x05_Pin, Connector_PinHeader_2.54mm:PinHeader_1x05_P2.54mm_Vertical, symbol Connector:Conn_01x05_Pin
- added J2, J4: Conn_01x05_Pin, Connector_PinHeader_2.54mm:PinHeader_1x05_P2.54mm_Horizontal, symbol Connector:Conn_01x05_Pin
- added JP1, JP2, JP3, JP4, JP5, JP6: Jumper_2_Bridged, TestPoint:TestPoint_2Pads_Pitch2.54mm_Drill0.8mm, symbol Jumper:Jumper_2_Bridged
Connections:
- net ADC2_offset is gone; now on net +1V65: A1.31 (MISO1/PA6)
- net +1V65: now also C18.1, J7.S, J8.S, J9.S; no longer J7.T, J8.T, J9.T
- net +3V3: no longer C17.1, C18.1
- net AC_C1: now also J7.T; no longer J7.S
- net AC_C2: now also J9.T; no longer J9.S
- net AC_C3: now also J8.T; no longer J8.S
- net AC_NEU: now also J4.4 (Pin_4), J4.5 (Pin_5)
- net AC_PH1: now also J4.1 (Pin_1), J4.2 (Pin_2)
- net GND: now also J2.4 (Pin_4), J2.5 (Pin_5)
- net RX_UART: now also J2.3 (Pin_3)
- net TX_UART: now also J2.2 (Pin_2)
- net +5V: now reaches A1.21 (VBAT)
- net +5V: now also C17.1, J2.1 (Pin_1)
- no-connect marks 6 -> 7
Other:
- note removed: "para una medición simultánea de los 2 ADC, se tiene que muestrear en la siguiente secuencia: V_PH1 -> CH0 en ADC1 y A_PH1 -> CH5 en ADC2 V_PH2 -> CH1 en ADC1 y A_PH2 -> CH4 en ADC2 V_PH3 -> CH2 en ADC1 y A_PH3 -> CH3 en ADC2"
- moved on the sheet: C15, C16, C17, J7, J8, J9, R10, R9, U6E, U7C, U7E

Commit message: branch completo-bicapa
Parts:
- removed J19, J20: Conn_01x05_Pin, Connector_PinHeader_2.54mm:PinHeader_1x05_P2.54mm_Vertical, symbol Connector:Conn_01x05_Pin
- removed J2, J4: Conn_01x05_Pin, Connector_PinHeader_2.54mm:PinHeader_1x05_P2.54mm_Horizontal, symbol Connector:Conn_01x05_Pin
- added C1: 100n, Capacitor_THT:CP_Radial_Tantal_D5.5mm_P2.50mm, symbol Device:C
- added C2: 10u, Capacitor_THT:CP_Radial_D6.3mm_P2.50mm, symbol PCM_Capacitor_AKL:CP_Generic
- added F1: Fuse, Fuse:Fuseholder_Clip-5x20mm_Littelfuse_445-030_Inline_P20.50x5.20mm_D1.30mm_Horizontal, symbol Device:Fuse
- added J2: Conn_01x12_Pin, Connector_PinHeader_2.54mm:PinHeader_1x12_P2.54mm_Vertical, symbol Connector:Conn_01x12_Pin
- added RV1: Varistor, Varistor:RV_Disc_D12mm_W3.9mm_P7.5mm, symbol Device:Varistor
- added U1: HLK-5M05, Converter_ACDC:Converter_ACDC_Hi-Link_HLK-5Mxx, symbol Converter_ACDC:HLK-5M05
- added U2: ESP32-C3-SuperMini, esp32-c3-supermini:ESP32-C3-SuperMini, symbol esp32-c3-supermini:ESP32-C3-SuperMini
- R12: value 820 -> 820k
- R13: value R -> 820k
- R17, R20: value R -> 3.3k
- R18, R19, R22: value R -> 10k
- R21: value 820 -> 10k
Connections:
- net +3V3: no longer A1.20 (3V3)
- net +5V: now also C1.1, C2.1, U1.4 (+Vout), U2.8 (5V)
- net AC_C1: now also JP4.1 (A); no longer U3.7 (P0B)
- net AC_C2: now also JP6.1 (A); no longer U5.7 (P0B)
- net AC_C3: now also JP5.1 (A); no longer U4.5 (P0A)
- net AC_PH1: now also J6.1 (Pin_1), F1.1; no longer J6.2 (Pin_2)
- net AC_PH2: now also J6.2 (Pin_2); no longer J6.3 (Pin_3)
- net AC_PH3: now also J6.3 (Pin_3); no longer J6.4 (Pin_4)
- net ADC2_CH3: now also U5.7 (P0B); no longer U5.5 (P0A)
- net ADC2_CH5: now also U3.7 (P0B); no longer U3.5 (P0A)
- net GND: now also C1.2, C2.2, J2.1 (Pin_1), J2.10 (Pin_10), J2.11 (Pin_11), J2.12 (Pin_12), J2.2 (Pin_2), J2.3 (Pin_3), J2.4 (Pin_4), J2.5 (Pin_5), J2.6 (Pin_6), J2.7 (Pin_7), J2.8 (Pin_8), J2.9 (Pin_9), U1.3 (-Vout), U2.7 (GND)
- net at J14.1 (Pin_1): now also JP5.2 (B), U4.5 (P0A)
- net at R17.2, TR2.4: now also JP2.1 (A); no longer R18.2
- net at J12.1 (Pin_1): now also JP3.2 (B), R21.2
- net at JP1.1 (A): now also R14.2, TR1.4
- net at JP1.2 (B): now also J5.1 (Pin_1), R15.2
- net at J11.1 (Pin_1): now also JP2.2 (B), R18.2
- net at J13.1 (Pin_1): now also JP4.2 (B), U3.5 (P0A)
- net at JP3.1 (A): now also R20.2, TR3.4
- net at JP6.2 (B): now also J18.1 (Pin_1), U5.5 (P0A)
- net AC_NEU renamed GNDPWR
- net GNDPWR: now also J6.4 (Pin_4), RV1.2, U1.2 (AC/N); no longer J6.1 (Pin_1)
- net RX_UART: no longer names the net of A1.15 (PB7/SDA1/RX1)
- net RX_UART: now also U2.16 (GPIO21)
- net TX_UART: no longer names the net of A1.14 (PB6/SCL1/TX1)
- net TX_UART: now also U2.15 (GPIO20)
- new net VAC: F1.2, RV1.1, U1.1 (AC/L)
- no-connect marks 7 -> 19
Other:
- note added: "Alimentación OpAmps"
- note added: "Conector Trifásico y Alimentación"
- note added: "Generación Voltaje de Referencia"
- note added: "Masas p/ Testeo"
- note added: "Montaje"
- note added: "Placa de Desarrollo ESP32-C3 + STM32F103"
- note added: "Sensado de Corriente"
- note added: "Sensado de Voltaje"
- moved on the sheet: A1, C15, C16, C17, C18, H1, H2, H3, H4, J1, J10, J11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

Commit message: branch completo-unicapa wip
Parts:
- removed C17: 100n, Capacitor_THT:CP_Radial_Tantal_D5.5mm_P2.50mm, symbol Device:C
Connections:
- net ADC2_CH3: now also U5.5 (P0A); no longer U5.7 (P0B)
- net GND: no longer A1.19 (GND)
- net at J18.1 (Pin_1), JP6.2 (B): now also U5.7 (P0B); no longer U5.5 (P0A)
- no-connect marks 19 -> 20

Commit message: completo unicapa
Parts:
- removed J2: Conn_01x12_Pin, Connector_PinHeader_2.54mm:PinHeader_1x12_P2.54mm_Vertical, symbol Connector:Conn_01x12_Pin
- added C19: 100n, Capacitor_THT:CP_Radial_Tantal_D5.5mm_P2.50mm, symbol Device:C
- added J19, J2, J20, J4: Conn_01x03_Pin, Connector_PinHeader_2.54mm:PinHeader_1x03_P2.54mm_Vertical, symbol Connector:Conn_01x03_Pin
Connections:
- net +1V65: now also C19.1
- net +5V: now also A1.18 (5V); no longer A1.21 (VBAT)
- net ADC2_CH3: now also U5.7 (P0B); no longer U5.5 (P0A)
- net GND: now also C19.2, J19.1 (Pin_1), J19.2 (Pin_2), J19.3 (Pin_3), J2.1 (Pin_1), J2.2 (Pin_2), J2.3 (Pin_3), J20.1 (Pin_1), J20.2 (Pin_2), J20.3 (Pin_3), J4.1 (Pin_1), J4.2 (Pin_2), J4.3 (Pin_3)
- net SPI_CS3: now also A1.33 (PB0); no longer A1.35 (SCL2/TX3/PB10)
- net SPI_CS5: now also A1.35 (SCL2/TX3/PB10); no longer A1.33 (PB0)
- net at J18.1 (Pin_1), JP6.2 (B): now also U5.5 (P0A); no longer U5.7 (P0B)
- no-connect marks 20 -> 21
Other:
- moved on the sheet: A1, C1, C15, C16, C18, C2, F1, H1, H2, H3, H4, J1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

Commit message: mejoras
Parts:
- added J21: Conn_01x02_Pin, Connector_Molex:Molex_KK-396_5273-02A_1x02_P3.96mm_Vertical, symbol Connector:Conn_01x02_Pin
- added J22: Conn_01x03_Pin, Connector_PinHeader_2.54mm:PinHeader_1x03_P2.54mm_Vertical, symbol Connector:Conn_01x03_Pin
Connections:
- net +5V: now also J21.1 (Pin_1)
- net AC_PH1: now also J6.2 (Pin_2); no longer J6.1 (Pin_1)
- net AC_PH2: now also J6.3 (Pin_3); no longer J6.2 (Pin_2)
- net AC_PH3: now also J6.4 (Pin_4); no longer J6.3 (Pin_3)
- net GND: now also A1.19 (GND), J21.2 (Pin_2), J22.3 (Pin_3)
- net GNDPWR: now also J6.1 (Pin_1); no longer J6.4 (Pin_4)
- net at A1.14 (PB6/SCL1/TX1), U2.15 (GPIO20): now also J22.1 (Pin_1)
- net at A1.15 (PB7/SDA1/RX1), U2.16 (GPIO21): now also J22.2 (Pin_2)
- no-connect marks 21 -> 20
Other:
- moved on the sheet: J6

Commit message: fix erc
Connections:
- net GNDPWR renamed AC_NEU
- net VAC: no longer names the net of F1.2, RV1.1, U1.1 (AC/L)
- no-connect marks 20 -> 39
Other:
- moved on the sheet: A1, F1, J22

Commit message: rev 2
Parts:
- removed J20: Conn_01x03_Pin, Connector_PinHeader_2.54mm:PinHeader_1x03_P2.54mm_Vertical, symbol Connector:Conn_01x03_Pin
- added J20: Conn_01x04_Pin, Connector_PinHeader_2.54mm:PinHeader_1x04_P2.54mm_Vertical, symbol Connector:Conn_01x04_Pin
- added J23: Conn_01x01_Pin, Connector_PinHeader_2.54mm:PinHeader_1x01_P2.54mm_Vertical, symbol Connector:Conn_01x01_Pin
Connections:
- net +1V65: now also J23.1 (Pin_1)
- net GND: now also J20.1 (Pin_1), J20.2 (Pin_2), J20.3 (Pin_3), J20.4 (Pin_4)
Changed lines of the file:
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@@
 	)
 	(junction
+		(at 246.38 171.45)
+		(diameter 0)
+		(color 0 0 0 0)
+	)
+	(junction
 		(at 247.65 237.49)
 		(diameter 0)
@@
 	)
 	(junction
+		(at 245.11 237.49)
+		(diameter 0)
+		(color 0 0 0 0)
+	)
+	(junction
 		(at 106.68 177.8)
 		(diameter 0)
@@
 	(wire
 		(pts
+			(xy 246.38 167.64) (xy 246.38 171.45)
+		)
+		(stroke
+			(width 0)
+			(type default)
+		)
+	)
+	(wire
+		(pts
 			(xy 129.54 40.64) (xy 129.54 43.18)
 		)
@@
 	(wire
 		(pts
+			(xy 245.11 237.49) (xy 247.65 237.49)
+		)
+		(stroke
+			(width 0)
+			(type default)
+		)
+	)
+	(wire
+		(pts
 			(xy 187.96 120.65) (xy 217.17 120.65)
 		)
@@
 	(wire
 		(pts
-			(xy 231.14 237.49) (xy 247.65 237.49)
+			(xy 231.14 237.49) (xy 245.11 237.49)
 		)
 		(stroke
@@
 	(wire
 		(pts
+			(xy 245.11 234.95) (xy 245.11 237.49)
+		)
+		(stroke
+			(width 0)
+			(type default)
+		)
+	)
+	(wire
+		(pts
 			(xy 129.54 35.56) (xy 118.11 35.56)
 		)
@@
 	)
 	(symbol
-		(lib_id "Connector:Conn_01x03_Pin")
-		(at 250.19 229.87 90)
-		(mirror x)
-		(unit 1)
-		(body_style 1)
-		(exclude_from_sim no)
-		(in_bom yes)
-		(on_board yes)
-		(in_pos_files yes)
-		(dnp no)
-		(property "Reference" "J20"
-			(at 250.19 224.79 90)
-			(show_name no)
-			(do_not_autoplace no)
-			(effects
-				(font
-					(size 1.27 1.27)
-				)
-			)
-		)
-		(property "Value" "Conn_01x03_Pin"
-			(at 250.19 227.33 90)
-			(show_name no)
-			(do_not_autoplace no)
-			(effects
-				(font
-					(size 1.27 1.27)
-				)
-			)
-		)
-		(property "Footprint" "Connector_PinHeader_2.54mm:PinHeader_1x03_P2.54mm_Vertical"
-			(at 250.19 229.87 0)
-			(hide yes)
-			(show_name no)
-			(do_not_autoplace no)
-			(effects
-				(font
-					(size 1.27 1.27)
-				)
-			)
-		)
-		(property "Datasheet" ""
-			(at 250.19 229.87 0)
-			(hide yes)
-			(show_name no)
-			(do_not_autoplace no)
-			(effects
-				(font
-					(size 1.27 1.27)
-				)
-			)
-		)
-		(property "Description" "Generic connector, single row, 01x03, script generated"
-			(at 250.19 229.87 0)
-			(hide yes)
-			(show_name no)
-			(do_not_autoplace no)
-			(effects
-				(font
-					(size 1.27 1.27)
-				)
-			)
-		)
-		(pin "1"
-		)
-		(pin "2"
-		)
-		(pin "3"
-		)
-		(instances
-			(project "kicad-pps"
-				(path "/3aaac0ed-0487-4b68-a13f-fe4577298336"
-					(reference "J20")
-					(unit 1)
-				)
-			)
-		)
-	)
-	(symbol
 		(lib_id "Jumper:Jumper_2_Bridged")
 		(at 196.85 45.72 0)
@@
 	)
 	(symbol
+		(lib_id "Connector:Conn_01x01_Pin")
+		(at 246.38 162.56 90)
+		(mirror x)
+		(unit 1)
+		(body_style 1)
+		(exclude_from_sim no)
+		(in_bom yes)
+		(on_board yes)
+		(in_pos_files yes)
+		(dnp no)
+		(property "Reference" "J23"
+			(at 245.11 161.9249 90)
+			(show_name no)
+			(do_not_autoplace no)
+			(effects
+				(font
+					(size 1.27 1.27)
+				)
+				(justify left)
+			)
+		)
+		(property "Value" "Conn_01x01_Pin"
+			(at 245.11 164.4649 90)
+			(show_name no)
+			(do_not_autoplace no)
+			(effects
+				(font
+					(size 1.27 1.27)
+				)
+				(justify left)
+			)
+		)
+		(property "Footprint" "Connector_PinHeader_2.54mm:PinHeader_1x01_P2.54mm_Vertical"
+			(at 246.38 162.56 0)
+			(hide yes)
+			(show_name no)
+			(do_not_autoplace no)
+			(effects
+				(font
+					(size 1.27 1.27)
+				)
+			)
+		)
+		(property "Datasheet" ""
+			(at 246.38 162.56 0)
+			(hide yes)
+			(show_name no)
+			(do_not_autoplace no)
+			(effects
+				(font
+					(size 1.27 1.27)
+				)
+			)
+		)
+		(property "Description" "Generic connector, single row, 01x01, script generated"
+			(at 246.38 162.56 0)
+			(hide yes)
+			(show_name no)
+			(do_not_autoplace no)
+			(effects
+				(font
+					(size 1.27 1.27)
+				)
+			)
+		)
+		(pin "1"
+		)
+		(instances
+			(project "kicad-pps"
+				(path "/3aaac0ed-0487-4b68-a13f-fe4577298336"
+					(reference "J23")
+					(unit 1)
+				)
+			)
+		)
+	)
+	(symbol
 		(lib_id "Amplifier_Operational:LMV324")
 		(at 340.36 107.95 0)
@@
 					(unit 1)
 				)
+			)
+		)
+	)
+	(symbol
+		(lib_id "Connector:Conn_01x04_Pin")
+		(at 247.65 229.87 90)
+		(mirror x)
+		(unit 1)
+		(body_style 1)
+		(exclude_from_sim no)
+		(in_bom yes)
+		(on_board yes)
+		(in_pos_files yes)
+		(dnp no)
+		(fields_autoplaced yes)
+		(property "Reference" "J20"
+			(at 248.92 224.79 90)
+			(show_name no)
+			(do_not_autoplace no)
+			(effects
+				(font
+					(size 1.27 1.27)
+				)
+			)
+		)
+		(property "Value" "Conn_01x04_Pin"
+			(at 248.92 227.33 90)
+			(show_name no)
+			(do_not_autoplace no)
+			(effects
+				(font
+					(size 1.27 1.27)
+				)
+			)
+		)
+		(property "Footprint" "Connector_PinHeader_2.54mm:PinHeader_1x04_P2.54mm_Vertical"
+			(at 247.65 229.87 0)
+			(hide yes)
+			(show_name no)
+			(do_not_autoplace no)
+			(effects
+				(font
+					(size 1.27 1.27)
+				)
+			)
+		)
+		(property "Datasheet" ""
+			(at 247.65 229.87 0)
+			(hide yes)
+			(show_name no)
+			(do_not_autoplace no)
+			(effects
+				(font
+					(size 1.27 1.27)
+				)
+			)
+		)
+		(property "Description" "Generic connector, single row, 01x04, script generated"
+			(at 247.65 229.87 0)
+			(hide yes)
+			(show_name no)
+			(do_not_autoplace no)
+			(effects
+				(font
+					(size 1.27 1.27)
+				)
+			)
+		)
+		(pin "1"
+		)
+		(pin "2"
+		)
+		(pin "3"
+		)
+		(pin "4"
+		)
+		(instances
+			(project "kicad-pps"
+				(path "/3aaac0ed-0487-4b68-a13f-fe4577298336"
+					(reference "J20")
+					(unit 1)
+				)
